Commit message: Updated launch and urdf to include Kuka

File: urdf/demo.xacro (robot description, xacro)
@@ -3,8 +3,14 @@
   <xacro:arg name="use_mesh" default="true" />
   <!-- ur3 -->
-  <xacro:include filename="$(find ur_description)/urdf/inc/ur3_macro.xacro" />
+  <xacro:include filename="$(find iiwa_description)/urdf/iiwa7.xacro" />
   <xacro:include filename="$(find realsense2_description)/urdf/_d435.urdf.xacro" />
-  <!-- arm -->
-  <xacro:ur3_robot prefix=""/>
+  <!-- ROBOTS -->
+  <!--iiwa-->
+  <xacro:arg name="iiwa_hardware_interface" default="PositionJointInterface"/>
+  <xacro:iiwa7 hardware_interface="$(arg iiwa_hardware_interface)"
+               robot_name="iiwa"
+               parent="table">
+  <origin xyz="0.214 -0.324 0.50" rpy="0 0 1.63"/>
+  </xacro:iiwa7>
   <!-- camera -->
   <xacro:sensor_d435 parent="realsense_visual" use_nominal_extrinsics="$(arg use_nominal_extrinsics)" add_plug="$(arg add_plug)" use_mesh="$(arg use_mesh)">
@@ -22,5 +28,5 @@
   </link>
   <joint name="tool_to_aluminum" type="fixed">
-    <parent link="tool0"/>
+    <parent link="iiwa_link_ee"/>
     <child link="realsense_visual"/>
     <origin xyz="-0.04 0.0 0.0" rpy="0 0 0"/>
@@ -47,9 +53,9 @@
     <origin xyz="0.0 0.0 0.0" rpy="0.0 0.0 0.0" />
   </joint>
-  <joint name="table_to_base_link_joint" type="fixed">
+  <!-- <joint name="table_to_base_link_joint" type="fixed">
     <parent link="table" />
     <child link = "base_link" />
     <origin xyz="0.6 0.0 0.5" rpy="0.0 0.0 0.0" />
-  </joint>
+  </joint> -->
   <!-- realsense calibration stuff -->
   <link name="camera_color_optical_frame_x_trans"/>
@@ -60,5 +66,5 @@
   <link name="camera_color_optical_frame"/>
   <joint name="camera_color_optical_frame_x_joint" type="prismatic">
-    <parent link="tool0"/>
+    <parent link="iiwa_link_ee"/>
     <child link="camera_color_optical_frame_x_trans"/>
     <origin rpy="0 0 0" xyz="0 0 0"/>

Commit message: Updated to include iiwa hardware and fixed capture

File: urdf/demo.xacro (robot description, xacro)
@@ -2,18 +2,24 @@
   <xacro:arg name="add_plug" default="false" />
   <xacro:arg name="use_mesh" default="true" />
-  <!-- ur3 -->
+  <material name="Grey">
+    <color rgba="0.4 0.4 0.4 1.0"/>
+  </material>
+  <material name="Orange">
+    <color rgba="${255/255} ${108/255} ${10/255} 1.0"/>
+  </material>
+  <!-- iiwa7 -->
   <xacro:include filename="$(find iiwa_description)/urdf/iiwa7.xacro" />
   <xacro:include filename="$(find realsense2_description)/urdf/_d435.urdf.xacro" />
   <!-- ROBOTS -->
-  <!--iiwa-->
+  <!--iiwa7-->
   <xacro:arg name="iiwa_hardware_interface" default="PositionJointInterface"/>
   <xacro:iiwa7 hardware_interface="$(arg iiwa_hardware_interface)"
                robot_name="iiwa"
                parent="table">
-  <origin xyz="0.214 -0.324 0.50" rpy="0 0 1.63"/>
+    <origin xyz="0.8 0.0 0.50" rpy="0 0 1.57"/>
   </xacro:iiwa7>
   <!-- camera -->
   <xacro:sensor_d435 parent="realsense_visual" use_nominal_extrinsics="$(arg use_nominal_extrinsics)" add_plug="$(arg add_plug)" use_mesh="$(arg use_mesh)">
-    <origin xyz="0 0 0" rpy="0 0 0"/>
+    <origin xyz="-0.05 0 .0125" rpy="0 -1.57 0"/>
   </xacro:sensor_d435>
   <link name="realsense_visual">

Commit message: Updated with camera calibration files

File: urdf/demo.xacro (robot description, xacro)
@@ -65,10 +65,16 @@
   </joint> -->
   <!-- realsense calibration stuff -->
-  <link name="camera_color_optical_frame_x_trans"/>
+  <link name="camera_color_optical_frame"/>
+  <joint name="calib_camera_joint" type="fixed">
+    <parent link="iiwa_link_ee"/>
+    <child link="camera_color_optical_frame"/>
+    <origin rpy="-3.13477 -3.13857 1.57876" xyz="-0.0762939 0.00946182 0.0607092" />
+  </joint>
+  <!-- <link name="camera_color_optical_frame_x_trans"/>
   <link name="camera_color_optical_frame_y_trans"/>
   <link name="camera_color_optical_frame_z_trans"/>
   <link name="camera_color_optical_frame_pitch"/>
-  <link name="camera_color_optical_frame_yaw"/>
-  <link name="camera_color_optical_frame"/>
+  <link name="camera_color_optical_frame_yaw"/> -->
+<!--
   <joint name="camera_color_optical_frame_x_joint" type="prismatic">
     <parent link="iiwa_link_ee"/>
@@ -112,7 +118,7 @@
     <limit effort="2" lower="-6.2832" upper="6.2832" velocity="10"/>
     <axis xyz="1 0 0"/>
-  </joint>
+  </joint> -->
   <!-- target calibration stuff -->
-  <link name="target"/>
+  <!-- <link name="target"/>
   <link name="target_x_trans">
     <visual>
@@ -168,10 +174,10 @@
     <limit effort="2" lower="-6.2832" upper="6.2832" velocity="10"/>
     <axis xyz="1 0 0"/>
-  </joint>
+  </joint> -->
   <link name="target_calibrated"/>
   <joint name="target_calibrated_joint" type="fixed">
-    <parent link="world"/>
+    <parent link="iiwa_link_0"/>
     <child link="target_calibrated"/>
-    <origin rpy="-1.5712 0.0098 0.0073" xyz="0.5242 0.2895 0.5130"/>
+    <origin rpy="-3.14145 3.13462 1.56692" xyz="-0.20862 0.595346 0.00766619"/>
   </joint>
 </robot>

Commit message: updated paths for the scannig

File: urdf/demo.xacro (robot description, xacro)
@@ -69,5 +69,5 @@
     <parent link="iiwa_link_ee"/>
     <child link="camera_color_optical_frame"/>
-    <origin rpy="-3.13477 -3.13857 1.57876" xyz="-0.0762939 0.00946182 0.0607092" />
+    <origin rpy="-3.13573 -3.13968 1.5879" xyz="-0.0760461 -0.0123072 0.05901180" />
   </joint>
   <!-- <link name="camera_color_optical_frame_x_trans"/>
@@ -179,5 +179,5 @@
     <parent link="iiwa_link_0"/>
     <child link="target_calibrated"/>
-    <origin rpy="-3.14145 3.13462 1.56692" xyz="-0.20862 0.595346 0.00766619"/>
+    <origin rpy="0.122741 0.01472 3.10858" xyz="0.0425594 -0.569619 -0.159719"/>
   </joint>
 </robot>
